Commit message: Update baselink

File: wamv_gazebo/urdf/components/wamv_gps.xacro (robot description, xacro)
@@ -31,5 +31,5 @@
       <limit effort="1000.0" lower="0.0" upper="0" velocity="0"/>
       <origin xyz="${x} ${y} ${z}" rpy="${R} ${P} ${Y}" />
-      <parent link="${namespace}/base_link" />
+      <parent link="base_link" />
       <child link="${namespace}/${name}_link" />
     </joint>

File: wamv_gazebo/urdf/components/wamv_imu.xacro (robot description, xacro)
@@ -20,5 +20,5 @@
       <limit effort="1000.0" lower="0.0" upper="0" velocity="0"/>
       <origin xyz="${x} ${y} ${z}" rpy="${R} ${P} ${Y}"/>
-      <parent link="${namespace}/base_link"/>
+      <parent link="base_link"/>
       <child link="${namespace}/${name}_link"/>
     </joint>
